File: FeatherWing.sch (EAGLE design)
At the start: 9 parts, among them X2 LEDMATRIXFPCCONNECTOR_CON-HIR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, X3 REMBRANDT-ELECTRONICS---JST-X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, X4 REMBRANDT-ELECTRONICS---JST-X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

Commit message: pi HAT with preipherals for the office project need
Changed lines of the file:
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@@
 <wire x1="288.036" y1="85.09" x2="288.036" y2="88.9" width="0.1524" layer="91"/>
 <wire x1="288.036" y1="88.9" x2="292.1" y2="88.9" width="0.1524" layer="91"/>
-<label x="292.1" y="88.9" size="1.27" layer="95" rot="R180" xref="yes"/>
+<label x="292.1" y="88.9" size="1.27" layer="95" xref="yes"/>
 </segment>
 </net>
